Commit message: adjust joint limits

File: config/spot.urdf (robot description, URDF)
Before this commit: robot spot, 24 links, 23 joints
Links:
- added link hand
Joints:
- added joint arm_wr1_to_hand: type fixed, parent arm_link_wr1, child hand, origin xyz=0.19557 0 0 rpy=0 0 0

Commit message: Use saved sensor mount geometry in MoveIt

File: config/spot.urdf (robot description, URDF)
Before this commit: robot spot, 25 links, 24 joints
Links:
- added link sensor_head_slot
- link arm_link_wr1: geometry collision mesh filename=package://spot_description/meshes/arm/collision/arm_link_wr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; visual mesh filename=package://spot_description/meshes/arm/visual/arm_link_wr1.o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
Joints:
- added joint hand_to_sensor_head_slot: type fixed, parent hand, child sensor_head_slot, origin xyz=0 0 0 rpy=0 0 0

Commit message: add collision geometry

File: config/spot.urdf (robot description, URDF)
Before this commit: robot spot, 26 links, 25 joints
Links:
- link arm_link_hr0: geometry collision mesh filename=package://spot_moveit_config/config/collision/arm_link_hr0.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; visual mesh filename=package://spot_description/meshes/arm/visual/arm_link_hr0.o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
- link front_left_hip: geometry collision mesh filename=package://spot_moveit_config/config/collision/front_left_hi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; visual mesh filename=package://spot_description/meshes/base/visual/front_left_hi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
- link front_right_hip: geometry collision mesh filename=package://spot_moveit_config/config/collision/front_right_h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; visual mesh filename=package://spot_description/meshes/base/visual/front_right_h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
- link rear_left_hip: geometry collision mesh filename=package://spot_moveit_config/config/collision/rear_left_hip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; visual mesh filename=package://spot_description/meshes/base/visual/rear_left_hip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
- link rear_right_hip: geometry collision mesh filename=package://spot_moveit_config/config/collision/rear_right_hi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; visual mesh filename=package://spot_description/meshes/base/visual/rear_right_hi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
